Commit message: edited launch files

File: gazebo_simulation/turtlebot_description/urdf/lidar.xacro (robot description, xacro)
@@ -2,16 +2,4 @@
     <xacro:macro name="rplidar">
         <link name="laser"/>
-            <!-- <visual>
-                <origin xyz="0 0 0" rpy="-1.5708 0 -1.5708"/>
-                <geometry>
-                    <mesh filename="file://$(find turtlebot_description)/meshes/HC-SR04.stl" scale="0.001 0.001 0.001"/>
-                </geometry>
-            </visual>
-            <collision>
-                <origin xyz="0 0 0" rpy="-1.5708 0 -1.5708"/>
-                <geometry>
-                    <mesh filename="file://$(find turtlebot_description)/meshes/HC-SR04.stl" scale="0.001 0.001 0.001"/>
-                </geometry>
-            </collision> -->
         <joint name="lidar_joint" type="fixed">
             <origin xyz = "0 0 0.1"/>
